Commit message: update files

File: src/lab2andDriver/drivers/universal_robot/ur_description/urdf/ur3.urdf (copy).xacro (robot description, xacro)
@@ -335,19 +335,12 @@
       <material>Gazebo/Grey</material>
     </gazebo>
-    <link name="${prefix}Screw_gripper">
+    <link name="${prefix}vacuum_gripper">
       <gravity>0</gravity>
       <visual>
         <origin rpy="0 0 0" xyz="0 0 0"/>
         <geometry>
-          <!-- <cylinder radius="0.005" length="0.01"/> -->
-          <mesh filename="package://ur_description/meshes/ur3/visual/Screw_Gripper.dae" scale="1 1 1"/>
-        </geometry>
-      </visual>
-      <collision>
-        <geometry>
-          <!-- <cylinder radius="0.005" length="0.01"/> -->
-          <mesh filename="package://ur_description/meshes/ur3/collision/Screw_Gripper.dae"/>
-        </geometry>
-      </collision>
+          <cylinder radius="0.005" length="0.01"/>
+        </geometry>
+      </visual>
       <inertial>
         <origin rpy="0 0 0" xyz="0.000000 0.000000 0.000000"/>
@@ -356,39 +349,19 @@
       </inertial>
     </link>
-    <gazebo reference="${prefix}Screw_gripper">
-        <material name="ChassisRed">
-          <color rgba="0.851 0.0 0.0 1.0"/>
-        </material>
+    <gazebo reference="${prefix}vacuum_gripper">
+      <material>Gazebo/Black</material>
     </gazebo>
     <joint name="${prefix}gripper_joint" type="revolute">
       <axis xyz="1 0 0" />
       <parent link="${prefix}ee_link" />
-      <child link="${prefix}Screw_gripper" />
-      <!-- <origin rpy="0 1.5708 0" xyz="0.059 0.0535 0" /> -->
+      <child link="${prefix}vacuum_gripper" />
       <origin rpy="0 1.5708 0" xyz="0.059 0.0535 0" />
       <limit effort="50" velocity="50" lower="0" upper="0" />
       <dynamics damping="0.0" friction="10"/>
     </joint>
-    <transmission name="gripper_tran"><!-- 名字自定义  -->
-      <type>transmission_interface/SimpleTransmission</type>
-      <joint name="${prefix}gripper_joint"><!-- 名字必须与swivel_J0对应一致  -->
-        <hardwareInterface>EffortJointInterface</hardwareInterface>
-      </joint>
-      <actuator name="gripper_motor"><!-- 名字自定义  -->
-        <hardwareInterface>EffortJointInterface</hardwareInterface>
-        <mechanicalReduction>1</mechanicalReduction>
-      </actuator>
-    </transmission>
     <gazebo>
-      <plugin name="gazebo_ros_control" filename="libgazebo_ros_control.so">
-        <robotNamespace>/gripper</robotNamespace>
-        <controlPeriod>0.01</controlPeriod>
-        <robotSimType>gazebo_ros_control/DefaultRobotHWSim</robotSimType>
-      </plugin>
-    </gazebo>
-    <!-- <gazebo>
       <plugin name="gazebo_ros_vacuum_gripper" filename="libgazebo_ros_vacuum_gripper.so">
         <robotNamespace>/gripper</robotNamespace>
-        <bodyName>${prefix}Screw_gripper</bodyName>
+        <bodyName>${prefix}vacuum_gripper</bodyName>
         <topicName>grasping</topicName>
         <maxForce>0.5</maxForce>
@@ -396,5 +369,5 @@
         <minDistance>0.01</minDistance>
       </plugin>
-    </gazebo> -->
+    </gazebo>
     <xacro:ur_arm_transmission prefix="${prefix}" hw_interface="${transmission_hw_interface}" />
     <xacro:ur_arm_gazebo prefix="${prefix}" />
