Commit message: project update 2 final version

File: src/lab2andDriver/drivers/universal_robot/ur_description/urdf/block_largerHole.urdf (robot description, URDF)
Before this commit: robot block_largerHole, 1 links, 0 joints
Links:
- added link world
Joints:
- added joint fixed: type fixed, parent world, child base_link

File: src/lab2andDriver/drivers/universal_robot/ur_description/urdf/screw_M8.urdf (robot description, URDF)
Before this commit: robot screw_M8, 1 links, 0 joints
Links:
- link base_link: mass 0.0001 -> 0.004

File: src/lab2andDriver/drivers/universal_robot/ur_description/urdf/ur3.urdf.xacro (robot description, xacro)
@@ -335,18 +335,18 @@
       <material>Gazebo/Grey</material>
     </gazebo>
-    <link name="${prefix}Screw_gripper">
+    <link name="${prefix}vacuum_gripper">
       <gravity>0</gravity>
       <visual>
         <origin rpy="0 0 0" xyz="0 0 0"/>
         <geometry>
-          <!-- <cylinder radius="0.005" length="0.01"/> -->
+          <!-- <cylinder radius="0.0025" length="0.01"/> -->
           <mesh filename="package://ur_description/meshes/ur3/visual/Screw_Gripper.dae" scale="1 1 1"/>
         </geometry>
       </visual>
-      <collision>
+      <!-- <collision>
         <geometry>
           <mesh filename="package://ur_description/meshes/ur3/visual/Screw_Gripper.dae"/>
         </geometry>
-      </collision>
+      </collision> -->
       <inertial>
         <origin rpy="0 0 0" xyz="0.000000 0.000000 0.000000"/>
@@ -355,15 +355,13 @@
       </inertial>
     </link>
-    <gazebo reference="${prefix}Screw_gripper">
-        <material name="ChassisRed">
-          <color rgba="0.851 0.0 0.0 1.0"/>
-        </material>
+    <gazebo reference="${prefix}vacuum_gripper">
+        <material>Gazebo/White</material>
     </gazebo>
     <joint name="${prefix}gripper_joint" type="revolute">
       <axis xyz="1 0 0" />
       <parent link="${prefix}ee_link" />
-      <child link="${prefix}Screw_gripper" />
+      <child link="${prefix}vacuum_gripper" />
       <origin rpy="0 1.5708 0" xyz="0.059 0.0535 0" />
-      <limit effort="50" velocity="50" lower="0" upper="0" />
+      <limit effort="10" velocity="0.01" lower="0" upper="0" />
       <dynamics damping="0.0" friction="10"/>
     </joint>
@@ -371,5 +369,5 @@
       <plugin name="gazebo_ros_vacuum_gripper" filename="libgazebo_ros_vacuum_gripper.so">
         <robotNamespace>/gripper</robotNamespace>
-        <bodyName>${prefix}Screw_gripper</bodyName>
+        <bodyName>${prefix}vacuum_gripper</bodyName>
         <topicName>grasping</topicName>
         <maxForce>0.5</maxForce>
