Commit message: project update2 finalize

File: src/lab2andDriver/drivers/universal_robot/ur_description/urdf/ur3.urdf.xacro (robot description, xacro)
@@ -335,12 +335,18 @@
       <material>Gazebo/Grey</material>
     </gazebo>
-    <link name="${prefix}vacuum_gripper">
+    <link name="${prefix}Screw_gripper">
       <gravity>0</gravity>
       <visual>
         <origin rpy="0 0 0" xyz="0 0 0"/>
         <geometry>
-          <cylinder radius="0.005" length="0.01"/>
-        </geometry>
-      </visual>
+          <!-- <cylinder radius="0.005" length="0.01"/> -->
+          <mesh filename="package://ur_description/meshes/ur3/visual/Screw_Gripper.dae" scale="1 1 1"/>
+        </geometry>
+      </visual>
+      <collision>
+        <geometry>
+          <mesh filename="package://ur_description/meshes/ur3/visual/Screw_Gripper.dae"/>
+        </geometry>
+      </collision>
       <inertial>
         <origin rpy="0 0 0" xyz="0.000000 0.000000 0.000000"/>
@@ -349,11 +355,13 @@
       </inertial>
     </link>
-    <gazebo reference="${prefix}vacuum_gripper">
-      <material>Gazebo/Black</material>
+    <gazebo reference="${prefix}Screw_gripper">
+        <material name="ChassisRed">
+          <color rgba="0.851 0.0 0.0 1.0"/>
+        </material>
     </gazebo>
     <joint name="${prefix}gripper_joint" type="revolute">
       <axis xyz="1 0 0" />
       <parent link="${prefix}ee_link" />
-      <child link="${prefix}vacuum_gripper" />
+      <child link="${prefix}Screw_gripper" />
       <origin rpy="0 1.5708 0" xyz="0.059 0.0535 0" />
       <limit effort="50" velocity="50" lower="0" upper="0" />
@@ -363,5 +371,5 @@
       <plugin name="gazebo_ros_vacuum_gripper" filename="libgazebo_ros_vacuum_gripper.so">
         <robotNamespace>/gripper</robotNamespace>
-        <bodyName>${prefix}vacuum_gripper</bodyName>
+        <bodyName>${prefix}Screw_gripper</bodyName>
         <topicName>grasping</topicName>
         <maxForce>0.5</maxForce>

Commit message: change end-effector color

File: src/lab2andDriver/drivers/universal_robot/ur_description/urdf/ur3.urdf.xacro (robot description, xacro)
@@ -333,5 +333,5 @@
     </link>
     <gazebo reference="${prefix}ee_link">
-      <material>Gazebo/Grey</material>
+      <material>Gazebo/Yellow</material>
     </gazebo>
     <link name="${prefix}vacuum_gripper">

Commit message: picking and driving screws

File: src/lab2andDriver/drivers/universal_robot/ur_description/urdf/ur3.urdf.xacro (robot description, xacro)
@@ -340,6 +340,6 @@
         <origin rpy="0 0 0" xyz="0 0 0"/>
         <geometry>
-          <!-- <cylinder radius="0.0025" length="0.01"/> -->
-          <mesh filename="package://ur_description/meshes/ur3/visual/Screw_Gripper.dae" scale="1 1 1"/>
+          <cylinder radius="0.0025" length="0.01"/>
+          <!-- <mesh filename="package://ur_description/meshes/ur3/visual/Screw_Gripper.dae" scale="1 1 1"/> -->
         </geometry>
       </visual>
