Commit message: human

File: src/lab2andDriver/drivers/universal_robot/ur_description/urdf/human.urdf (robot description, URDF)
Before this commit: robot Human, 2 links, 1 joints
Links:
- link base_link: geometry collision mesh filename=package://ur_description/meshes/ur3/collision/human.dae scale=0.1 0.1 0.1; visual mesh filename=package://ur_description/meshes/ur3/visual/human.dae scale=0.1 0.1 0.1
