Commit message: motion planning implementation

File: src/lab2andDriver/drivers/universal_robot/ur_description/urdf/blob.urdf (robot description, URDF)
Before this commit: robot block, 1 links, 0 joints
Links:
- link base_link: geometry collision cylinder length=0.03 radius=0.03; visual cylinder length=0.03 radius=0.03
